File: Hardware/PCB.brd (EAGLE design)
At the start: 46 x 35 mm, 105 parts, among them IC1 BQ25180YBGR, IC2 DRV2605YZFR, IC3 BMA423, IC9 RT6160AWSC, J1 TC2030-IDC, J2 503480-2400, J3 KH-TYPE-C-16P, Q1 20V/4.2A/52mΩ/1.4W, Q3 SI1308EDL-T1-GE3, U3 MAX17048G+T10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

Commit message: resolved all issues
Parts:
- moved C22 3.05 mm to (55.6, 152.9)
- moved ANT1 1.02 mm to (57.6, 154.6)
Connections:
- net N$11 renamed P0.00/XL1
- net N$12 renamed P0.01/XL2
Routing:
- net N$20: track 6.17 -> 7.47 mm
Other:
- outline, holes or cut-outs redrawn
